File: PCB Files/ESP32 PCB/ESP32 PCB.kicad_sch (KiCad schematic)
At the start: 36 parts, among them U1 Electrodes, U2 Electrodes, U3 LM324, U5 AHT20

Commit message: Update
Parts:
- C1: value (none) -> 2.7pF; footprint (none) -> Capacitor_SMD:C_1206_3216Metric
- C10, C6: value (none) -> 0.1uF; footprint (none) -> Capacitor_SMD:C_1206_3216Metric
- C2: value (none) -> 4.7pF; footprint (none) -> Capacitor_SMD:C_1206_3216Metric
- C9: value (none) -> 10uF; footprint (none) -> Capacitor_SMD:C_1206_3216Metric
- E1: value (none) -> PRO-OB-440; footprint (none) -> Antenna:ANT_PRO-OB-440
- J1: value (none) -> Conn_01x02; footprint (none) -> Connector_PinHeader_2.54mm:PinHeader_1x02_P2.54mm_Vertical
- L1: value (none) -> 1.6nH; footprint (none) -> Inductor_SMD:L_0805_2012Metric_Pad1.15x1.40mm_HandSolder
- R4, R5: value (none) -> 10K; footprint (none) -> Resistor_SMD:R_1206_3216Metric_Pad1.30x1.75mm_HandSolder
- TP1, TP2, TP3, TP4: value (none) -> TestPoint; footprint (none) -> TestPoint:TestPoint_Pad_D1.5mm
- U4: value (none) -> ESP32-PICO-D4; footprint (none) -> ESP_32:PQFN50P700X700X104-49N
Other:
- note added: "MCU"
- moved on the sheet: C10, C12, C14, C3, C4, C5, C7, C8, C9, J1, R1, R2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
