File: PCB Files/GSR + ST V2/GSR + ST V2.kicad_pcb (KiCad board)
At the start: 2 copper layers, 45.4 x 17.6 mm, 28 parts, among them J1 Conn_01x03, J2 Conn_01x02, U1 Electrodes, U2 Electrodes, U3 LM324, U4 AHT20

Commit message: Update
Parts:
- moved C5 0.81 mm to (212.0, 109.6)
- moved C7 0.10 mm to (211.9, 119.8)
- moved TP3 0.10 mm to (210.5, 107.1)
Routing:
- net Net-(R4-Pad1): track 20.9 -> 18.2 mm
- net Net-(J2-Pad1): track 28.0 -> 29.9 mm
- net Net-(C3-Pad2): track 27.0 -> 28.4 mm
- net Net-(C7-Pad1): track 34.0 -> 33.1 mm
- net +3V3: track 53.7 -> 53.2 mm
- net Net-(C8-Pad1): track 25.0 -> 25.5 mm
- net GND: vias 35 -> 32
