File: PCB Files/GSR + ST V2/GSR + ST V2.kicad_sch (KiCad schematic)
At the start: 26 parts, among them J1 Conn_01x03, J2 Conn_01x02, U1 Electrodes, U2 Electrodes, U3 LM324, U4 AHT20

Commit message: Update
Parts:
- C9: value 0.1uF -> (none)
Changed lines of the file:
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@@
       (effects (font (size 1.27 1.27)) (justify left))
     )
-    (property "Value" "0.1uF" (id 1) (at 106.68 119.3799 0)
+    (property "Value" "" (id 1) (at 106.68 119.3799 0)
       (effects (font (size 1.27 1.27)) (justify left))
     )
@@
     )
     (path "/df1435bb-8018-455d-9925-63e774164119"
-      (reference "C9") (unit 1) (value "0.1uF") (footprint "Capacitor_SMD:C_1206_3216Metric")
+      (reference "C9") (unit 1) (value "100nF") (footprint "Capacitor_SMD:C_1206_3216Metric")
     )
     (path "/59142adb-6887-41fc-851e-9a7f51511d60"
